File: MainBoard.brd (EAGLE design)
At the start: 160 x 106.3 mm, 47 parts, among them J37 POWER_JACKPTH_BREAD, U13 V_REG_317DPACK, U14 BQ27441-G1, U19 BQ24075

Commit message: Mainboard 1.1
Modified for 3 Door sensors
Parts:
- removed J30: (no value), SparkFun-Connectors:JST-3-PTH
- added J1, J4, J7: (no value), SparkFun-Connectors:JST-2-PTH
- added R10, R3, R9: 100k, SparkFun-Resistors:0603-RES@1
Connections:
- new net N$20: B1.29, J7.1, R3.1
- new net N$21: B1.30, J4.1, R9.1
- net GND: now also R10.2, R3.2, R9.2; no longer J30.1
- net GPOUT: no longer B1.31
- net N$81: now also B1.31, J1.1, R10.1; no longer J30.3
- net VCC: now also J1.2, J4.2, J7.2; no longer J30.2
Changed lines of the file:
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@@
 <attribute name="SF_ID" value="PRT-09915" x="1395.73" y="-364.49" size="1.778" layer="27" rot="R90" display="off"/>
-</element>
-<element name="J30" library="SparkFun-Connectors" package="JST-3-PTH" value="" x="154.94" y="34.29" rot="R90">
-<attribute name="PROD_ID" value="WIRE-10037" x="1412.24" y="-407.67" size="1.778" layer="27" rot="R90" display="off"/>
-<attribute name="SF_ID" value="PRT-09915" x="1412.24" y="-407.67" size="1.778" layer="27" rot="R90" display="off"/>
 </element>
 <element name="J37" library="SparkFun-Connectors" package="POWER_JACK_PTH_BREAD" value="POWER_JACKPTH_BREAD" x="2.54" y="93.98" rot="R270">
@@
 </element>
 <element name="JP11" library="SparkFun-Connectors" package="JST-2-SMD" value="" x="27.94" y="95.25">
-<attribute name="BTM_NEG" value="-" x="-604.52" y="-1315.72" size="1.778" layer="27" display="off"/>
-<attribute name="BTM_POS" value="+" x="-604.52" y="-1315.72" size="1.778" layer="27" display="off"/>
 <attribute name="PROD_ID" value="CONN-11443" x="-604.52" y="-1315.72" size="1.778" layer="27" display="off"/>
-<attribute name="TOP_NEG" value="-" x="-604.52" y="-1315.72" size="1.778" layer="27" display="off"/>
-<attribute name="TOP_POS" value="+" x="-604.52" y="-1315.72" size="1.778" layer="27" display="off"/>
+<attribute name="SF_ID" value="PRT-08612" x="27.94" y="95.25" size="1.778" layer="27" display="off"/>
 </element>
 <element name="C27" library="SparkFun-Capacitors" package="1206-CAP" value="1.0uF" x="17.78" y="81.28" rot="R90">
@@
 <attribute name="PROD_ID" value="CONN-08499" x="88.9" y="93.98" size="1.778" layer="27" display="off"/>
 <attribute name="SF_ID" value="PRT-0778" x="88.9" y="93.98" size="1.778" layer="27" display="off"/>
+</element>
+<element name="J1" library="SparkFun-Connectors" package="JST-2-PTH" value="" x="-12.7" y="-40.64">
+<attribute name="PROD_ID" value="CONN-09863" x="-12.7" y="-40.64" size="1.778" layer="27" display="off"/>
+<attribute name="SKU" value="PRT-09914" x="-12.7" y="-40.64" size="1.778" layer="27" display="off"/>
+</element>
+<element name="J4" library="SparkFun-Connectors" package="JST-2-PTH" value="" x="-12.7" y="-57.15">
+<attribute name="PROD_ID" value="CONN-09863" x="-12.7" y="-57.15" size="1.778" layer="27" display="off"/>
+<attribute name="SKU" value="PRT-09914" x="-12.7" y="-57.15" size="1.778" layer="27" display="off"/>
+</element>
+<element name="J7" library="SparkFun-Connectors" package="JST-2-PTH" value="" x="-12.7" y="-73.66">
+<attribute name="PROD_ID" value="CONN-09863" x="-12.7" y="-73.66" size="1.778" layer="27" display="off"/>
+<attribute name="SKU" value="PRT-09914" x="-12.7" y="-73.66" size="1.778" layer="27" display="off"/>
+</element>
+<element name="R9" library="SparkFun-Resistors" package="0603-RES@1" value="100k" x="-19.05" y="-189.23">
+<attribute name="PROD_ID" value="RES-00818" x="-19.05" y="-189.23" size="1.778" layer="27" display="off"/>
+</element>
+<element name="R10" library="SparkFun-Resistors" package="0603-RES@1" value="100k" x="-19.05" y="-193.04">
+<attribute name="PROD_ID" value="RES-00818" x="-19.05" y="-193.04" size="1.778" layer="27" display="off"/>
+</element>
+<element name="R3" library="SparkFun-Resistors" package="0603-RES@1" value="100k" x="-19.05" y="-196.85">
+<attribute name="PROD_ID" value="RES-00818" x="-19.05" y="-196.85" size="1.778" layer="27" display="off"/>
 </element>
 </elements>
@@
 <contactref element="J22" pad="1"/>
 <contactref element="J23" pad="1"/>
-<contactref element="J30" pad="1"/>
 <contactref element="C24" pad="-"/>
 <contactref element="R37" pad="1"/>
@@
 <wire x1="154.8384" y1="32.3088" x2="153.7716" y2="33.3756" width="0.1524" layer="1"/>
 <wire x1="142.3416" y1="33.3756" x2="142.24" y2="33.44" width="0.1524" layer="1"/>
-<wire x1="154.8384" y1="32.3088" x2="154.94" y2="32.29" width="0.1524" layer="1"/>
 <wire x1="128.016" y1="31.5468" x2="128.016" y2="24.2316" width="0.1524" layer="1"/>
 <wire x1="128.1684" y1="31.6992" x2="128.016" y2="31.5468" width="0.1524" layer="1"/>
@@
 <wire x1="154.9908" y1="32.3088" x2="156.0576" y2="33.3756" width="0.1524" layer="16"/>
 <wire x1="154.9908" y1="55.0164" x2="154.94" y2="55.15" width="0.1524" layer="16"/>
-<wire x1="154.9908" y1="32.3088" x2="154.94" y2="32.29" width="0.1524" layer="16"/>
 <wire x1="61.4172" y1="50.7492" x2="61.4172" y2="57.7596" width="0.1524" layer="16"/>
 <wire x1="77.8764" y1="34.29" x2="61.4172" y2="50.7492" width="0.1524" layer="16"/>
@@
 <wire x1="2.54" y1="86.36" x2="12.7" y2="86.36" width="0.1524" layer="1"/>
 <wire x1="12.7" y1="86.36" x2="13.3858" y2="87.0458" width="0.1524" layer="1"/>
+<contactref element="R10" pad="2"/>
+<contactref element="R9" pad="2"/>
+<contactref element="R3" pad="2"/>
+<wire x1="-18.2" y1="-193.04" x2="-18.2" y2="-196.85" width="0" layer="19" extent="1-1"/>
+<wire x1="-18.2" y1="-189.23" x2="-18.2" y2="-193.04" width="0" layer="19" extent="1-1"/>
+<wire x1="54.356" y1="2.54" x2="-18.2" y2="-189.23" width="0" layer="19" extent="1-1"/>
+<wire x1="154.9908" y1="32.3088" x2="154.8384" y2="32.3088" width="0" layer="19" extent="1-16"/>
 </signal>
 <signal name="VCC">
@@
 <contactref element="J22" pad="2"/>
 <contactref element="J23" pad="2"/>
-<contactref element="J30" pad="2"/>
 <contactref element="R36" pad="2"/>
 <contactref element="C25" pad="+"/>
@@
 <wire x1="154.8384" y1="34.29" x2="154.0764" y2="35.052" width="0.1524" layer="1"/>
 <wire x1="142.3416" y1="35.052" x2="142.24" y2="35.14" width="0.1524" layer="1"/>
-<wire x1="154.8384" y1="34.29" x2="154.94" y2="34.29" width="0.1524" layer="1"/>
 <wire x1="140.6652" y1="36.7284" x2="128.3208" y2="36.7284" width="0.1524" layer="1"/>
 <wire x1="142.1892" y1="35.2044" x2="140.6652" y2="36.7284" width="0.1524" layer="1"/>
@@
 <wire x1="152.4" y1="36.7284" x2="152.4" y2="46.6344" width="0.1524" layer="16"/>
 <wire x1="154.8384" y1="34.29" x2="152.4" y2="36.7284" width="0.1524" layer="16"/>
-<wire x1="154.8384" y1="34.29" x2="154.94" y2="34.29" width="0.1524" layer="16"/>
 <wire x1="76.0476" y1="34.8996" x2="62.7888" y2="48.1584" width="0.1524" layer="1"/>
 <wire x1="97.6884" y1="34.8996" x2="76.0476" y2="34.8996" width="0.1524" layer="1"/>
@@
 <wire x1="91.44" y1="96.6216" x2="91.44" y2="96.52" width="0.1524" layer="16"/>
 <via x="61.4172" y="97.0788" extent="1-16" drill="0.35"/>
+<contactref element="J4" pad="2"/>
+<contactref element="J1" pad="2"/>
+<contactref element="J7" pad="2"/>
+<wire x1="154.8384" y1="34.29" x2="154.8384" y2="34.29" width="0" layer="19" extent="1-16"/>
+<wire x1="-11.7" y1="-40.64" x2="76.0476" y2="34.8996" width="0" layer="19" extent="1-1"/>
+<wire x1="-11.7" y1="-57.15" x2="-11.7" y2="-40.64" width="0" layer="19" extent="1-1"/>
+<wire x1="-11.7" y1="-73.66" x2="-11.7" y2="-57.15" width="0" layer="19" extent="1-1"/>
 </signal>
 <signal name="N$8">
@@
 <signal name="N$81">
 <contactref element="B1" pad="28"/>
-<contactref element="J30" pad="3"/>
 <wire x1="154.8384" y1="42.2148" x2="154.8384" y2="36.4236" width="0.1524" layer="1"/>
 <wire x1="153.4668" y1="43.5864" x2="154.8384" y2="42.2148" width="0.1524" layer="1"/>
@@
 <wire x1="138.8364" y1="62.1792" x2="153.4668" y2="47.5488" width="0.1524" layer="1"/>
 <wire x1="128.3208" y1="62.1792" x2="138.8364" y2="62.1792" width="0.1524" layer="1"/>
-<wire x1="154.8384" y1="36.4236" x2="154.94" y2="36.29" width="0.1524" layer="1"/>
 <wire x1="128.3208" y1="62.1792" x2="128.27" y2="62.23" width="0.1524" layer="1"/>
+<contactref element="B1" pad="31"/>
+<contactref element="J1" pad="1"/>
+<contactref element="R10" pad="1"/>
+<wire x1="-13.7" y1="-40.64" x2="-19.9" y2="-193.04" width="0" layer="19" extent="1-1"/>
+<wire x1="128.27" y1="54.61" x2="-13.7" y2="-40.64" width="0" layer="19" extent="1-1"/>
+<wire x1="128.3208" y1="62.1792" x2="128.27" y2="54.61" width="0" layer="19" extent="1-1"/>
 </signal>
 <signal name="N$95">
@@
 <contactref element="R52" pad="1"/>
 <contactref element="U14" pad="12"/>
-<contactref element="B1" pad="31"/>
 <wire x1="59.7408" y1="64.3128" x2="62.7888" y2="64.3128" width="0.1524" layer="1"/>
 <wire x1="62.7888" y1="64.3128" x2="65.0748" y2="64.3128" width="0.1524" layer="1"/>
@@
 <wire x1="126.9492" y1="53.34" x2="105.0036" y2="53.34" width="0.1524" layer="1"/>
 <wire x1="128.1684" y1="54.5592" x2="126.9492" y2="53.34" width="0.1524" layer="1"/>
-<wire x1="128.1684" y1="54.5592" x2="128.27" y2="54.61" width="0.1524" layer="1"/>
 </signal>
 <signal name="TS">
@@
 <via x="110.0328" y="70.4088" extent="1-16" drill="0.35"/>
 </signal>
+<signal name="N$20">
+<contactref element="J7" pad="1"/>
+<contactref element="R3" pad="1"/>
+<contactref element="B1" pad="29"/>
+<wire x1="-13.7" y1="-73.66" x2="-19.9" y2="-196.85" width="0" layer="19" extent="1-1"/>
+<wire x1="128.27" y1="59.69" x2="-13.7" y2="-73.66" width="0" layer="19" extent="1-1"/>
+</signal>
+<signal name="N$21">
+<contactref element="J4" pad="1"/>
+<contactref element="R9" pad="1"/>
+<contactref element="B1" pad="30"/>
+<wire x1="-13.7" y1="-57.15" x2="-19.9" y2="-189.23" width="0" layer="19" extent="1-1"/>
+<wire x1="128.27" y1="57.15" x2="-13.7" y2="-57.15" width="0" layer="19" extent="1-1"/>
+</signal>
 </signals>
