File: MainBoard.sch (EAGLE design)
At the start: 47 parts, among them J37 POWER_JACKPTH_BREAD, U13 V_REG_317DPACK, U14 BQ27441-G1, U19 BQ24075

Commit message: Mainboard 1.1
Modified for 3 Door sensors
Parts:
- removed J30: (no value), SparkFun-Connectors:CONN_03JST-PTH
- added J1, J4, J7: (no value), SparkFun-Connectors:CONN_02JST-PTH-2
- added R10, R3, R9: 100k, SparkFun-Resistors:330OHM1/10W1%(0603)
Connections:
- new net N$20: B1.5, J7.1, R3.1
- new net N$21: B1.15, J4.1, R9.1
- net GND: now also R10.2, R3.2, R9.2; no longer J30.1
- net GPOUT: no longer B1.2
- net N$81: now also B1.2, J1.1, R10.1; no longer J30.3
- net VCC: now also J1.2, J4.2, J7.2; no longer J30.2
Other:
- moved on the sheet: BT1, BT2, BT3, C24, C25, C26, C27, C28, C29, C30, C55, D1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
